File: Adafruit QT Py.sch (EAGLE design)
At the start: 24 parts, among them IC3 ATSAMD21E, Q2 reset, U1 AP2112K-3.3, X6 USB TYPE C

Commit message: Update board files.
Parts:
- IC3: device microbuilder:ATSAMD21E -> adafruit_micro:ATSAMD21E
Connections:
- removed net CS: IC3.PA14/I14/SERCOM2+4.2, R1.2, U2.SSEL
- new net FLASH_CS: IC3.PA08/I2C/AIN16/SERCOM0+2.0/I2SD1, R1.2, U2.SSEL
- net MISO: now also IC3.PA09/I2C/I9/AIN17/SERCOM0+2.1/I2SMC; no longer IC3.PA10/I10/AIN18/SERCOM0+2.2/I2SCK
- net MISO2: now also IC3.PA19/I3/SERCOM1+3.3/I2SD0; no longer IC3.PA15/I15/SERCOM3+4.3
- net MOSI: now also IC3.PA10/I10/AIN18/SERCOM0+2.2/I2SCK; no longer IC3.PA08/I2C/AIN16/SERCOM0+2.0/I2SD1
- net NEOPIX: now also IC3.PA18/I2/SERCOM1+3.2; no longer IC3.PA19/I3/SERCOM1+3.3/I2SD0
- net NEO_PWR: now also IC3.PA15/I15/SERCOM2+4.3; no longer IC3.PA18/I2/SERCOM1+3.2
Other:
- moved on the sheet: R1
Changed lines of the file:
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@@
 <part name="GND14" library="supply1" library_urn="urn:adsk.eagle:library:371" deviceset="GND" device=""/>
 <part name="Q2" library="microbuilder" deviceset="SWITCH_TACT_SMT" device="4.6X2.8" value="reset"/>
-<part name="IC3" library="microbuilder" deviceset="ATSAMD21E" device=""/>
+<part name="IC3" library="adafruit_micro" deviceset="ATSAMD21E" device=""/>
 <part name="U$18" library="microbuilder" deviceset="3.3V" device=""/>
 <part name="GND18" library="supply1" library_urn="urn:adsk.eagle:library:371" deviceset="GND" device=""/>
@@
 <text x="132.08" y="154.94" size="1.778" layer="94">SERCOM0</text>
 <text x="129.54" y="124.46" size="1.778" layer="94">SERCOM1</text>
-<text x="132.08" y="147.32" size="1.778" layer="94">SERCOM2</text>
+<text x="129.54" y="142.24" size="1.778" layer="94">SERCOM2</text>
 <text x="129.54" y="106.68" size="1.778" layer="94">SERCOM3</text>
 </plain>
@@
 <attribute name="VALUE" x="24.384" y="34.036" size="1.27" layer="96" rot="R90"/>
 </instance>
-<instance part="R1" gate="G$1" x="132.08" y="132.08" smashed="yes" rot="R180">
-<attribute name="NAME" x="132.08" y="132.08" size="1.27" layer="95" font="vector" rot="R180" align="center"/>
-<attribute name="VALUE" x="132.08" y="129.54" size="1.016" layer="96" font="vector" ratio="15" rot="R180" align="center"/>
-</instance>
-<instance part="U$7" gate="G$1" x="137.16" y="134.62" smashed="yes">
-<attribute name="VALUE" x="135.636" y="135.636" size="1.27" layer="96"/>
+<instance part="R1" gate="G$1" x="142.24" y="149.86" smashed="yes" rot="R180">
+<attribute name="NAME" x="142.24" y="149.86" size="1.27" layer="95" font="vector" rot="R180" align="center"/>
+<attribute name="VALUE" x="142.24" y="147.32" size="1.016" layer="96" font="vector" ratio="15" rot="R180" align="center"/>
+</instance>
+<instance part="U$7" gate="G$1" x="152.4" y="147.32" smashed="yes" rot="R180">
+<attribute name="VALUE" x="153.924" y="146.304" size="1.27" layer="96" rot="R180"/>
 </instance>
 <instance part="TP1" gate="G$1" x="99.06" y="66.04" smashed="yes">
@@
 <pinref part="R1" gate="G$1" pin="1"/>
 <pinref part="U$7" gate="G$1" pin="3.3V"/>
+<wire x1="152.4" y1="149.86" x2="147.32" y2="149.86" width="0.1524" layer="91"/>
 </segment>
 </net>
@@
 </segment>
 <segment>
-<pinref part="IC3" gate="G$1" pin="PA08/I2C/AIN16/SERCOM0+2.0/I2SD1"/>
-<wire x1="114.3" y1="149.86" x2="127" y2="149.86" width="0.1524" layer="91"/>
-<label x="116.84" y="149.86" size="1.778" layer="95"/>
+<pinref part="IC3" gate="G$1" pin="PA10/I10/AIN18/SERCOM0+2.2/I2SCK"/>
+<wire x1="114.3" y1="144.78" x2="127" y2="144.78" width="0.1524" layer="91"/>
+<label x="116.84" y="144.78" size="1.778" layer="95"/>
 </segment>
 </net>
@@
 </segment>
 <segment>
-<pinref part="IC3" gate="G$1" pin="PA10/I10/AIN18/SERCOM0+2.2/I2SCK"/>
-<wire x1="114.3" y1="144.78" x2="127" y2="144.78" width="0.1524" layer="91"/>
-<label x="116.84" y="144.78" size="1.778" layer="95"/>
+<pinref part="IC3" gate="G$1" pin="PA09/I2C/I9/AIN17/SERCOM0+2.1/I2SMC"/>
+<wire x1="114.3" y1="147.32" x2="127" y2="147.32" width="0.1524" layer="91"/>
+<label x="116.84" y="147.32" size="1.778" layer="95"/>
 </segment>
 </net>
@@
 </segment>
 <segment>
-<pinref part="IC3" gate="G$1" pin="PA19/I3/SERCOM1+3.3/I2SD0"/>
-<wire x1="114.3" y1="119.38" x2="127" y2="119.38" width="0.1524" layer="91"/>
-<label x="116.84" y="119.38" size="1.778" layer="95"/>
+<pinref part="IC3" gate="G$1" pin="PA18/I2/SERCOM1+3.2"/>
+<wire x1="114.3" y1="121.92" x2="127" y2="121.92" width="0.1524" layer="91"/>
+<label x="116.84" y="121.92" size="1.778" layer="95"/>
 </segment>
 </net>
@@
 </segment>
 <segment>
-<pinref part="IC3" gate="G$1" pin="PA18/I2/SERCOM1+3.2"/>
-<wire x1="114.3" y1="121.92" x2="127" y2="121.92" width="0.1524" layer="91"/>
-<label x="116.84" y="121.92" size="1.778" layer="95"/>
+<pinref part="IC3" gate="G$1" pin="PA15/I15/SERCOM2+4.3"/>
+<wire x1="114.3" y1="129.54" x2="127" y2="129.54" width="0.1524" layer="91"/>
+<label x="116.84" y="129.54" size="1.778" layer="95"/>
 </segment>
 </net>
@@
 <net name="MISO2" class="0">
 <segment>
-<pinref part="IC3" gate="G$1" pin="PA15/I15/SERCOM3+4.3"/>
-<wire x1="114.3" y1="129.54" x2="127" y2="129.54" width="0.1524" layer="91"/>
-<label x="116.84" y="129.54" size="1.778" layer="95"/>
-</segment>
-<segment>
 <wire x1="25.4" y1="43.18" x2="22.86" y2="43.18" width="0.1524" layer="91"/>
 <pinref part="U2" gate="G$1" pin="MISO"/>
@@
 <label x="25.4" y="43.18" size="1.778" layer="95"/>
 </segment>
-</net>
-<net name="CS" class="0">
+<segment>
+<pinref part="IC3" gate="G$1" pin="PA19/I3/SERCOM1+3.3/I2SD0"/>
+<wire x1="114.3" y1="119.38" x2="127" y2="119.38" width="0.1524" layer="91"/>
+<label x="116.84" y="119.38" size="1.778" layer="95"/>
+</segment>
+</net>
+<net name="FLASH_CS" class="0">
 <segment>
 <pinref part="U2" gate="G$1" pin="SSEL"/>
@@
 </segment>
 <segment>
-<pinref part="IC3" gate="G$1" pin="PA14/I14/SERCOM2+4.2"/>
-<wire x1="114.3" y1="132.08" x2="127" y2="132.08" width="0.1524" layer="91"/>
-<label x="116.84" y="132.08" size="1.778" layer="95"/>
+<pinref part="IC3" gate="G$1" pin="PA08/I2C/AIN16/SERCOM0+2.0/I2SD1"/>
+<wire x1="114.3" y1="149.86" x2="137.16" y2="149.86" width="0.1524" layer="91"/>
+<label x="116.84" y="149.86" size="1.778" layer="95"/>
 <pinref part="R1" gate="G$1" pin="2"/>
 </segment>
